File: 1802-Mini-PIO.kicad_pcb (KiCad board)
At the start: 2 copper layers, 100 x 100 mm, 60 parts, among them J1 Mount, J10 OUT_PORTB, J11 INPUT, J12 OUTPUT_B, J13 OUTPUT_A, J2 Mount, J3 Mount, J4 Mount, J5 Expansion, J6 GRP_EXP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

Commit message: Finish Rev A board layout
Parts:
- moved J10 15.8 mm to (156.5, 89.1)
- moved J8 7.38 mm to (141.0, 89.1)
- moved J9 7.24 mm to (148.7, 89.1)
- moved JP1 5.06 mm to (191.0, 135.6), turned to 90 degrees
- moved C4 0.95 mm to (164.8, 99.5)
- moved C12 0.56 mm to (146.8, 70.1)
- moved U7 0.36 mm to (115.8, 71.4)
- moved C1 0.35 mm to (164.8, 137.6)
- moved C5 0.25 mm to (103.4, 109.7)
- moved U12 0.25 mm to (151.6, 71.4)
- moved C13 0.25 mm to (136.7, 129.2)
- moved C7 0.25 mm to (111.3, 70.1)
Routing:
- net GND: track 0.00 -> 507.9 mm
- net +5V: track 1.40 -> 442.9 mm
- net ~{EF4}: track 0.00 -> 148.2 mm
- net ~{EF3}: track 0.00 -> 134.0 mm
- net ~{CLEAR}: track 0.00 -> 124.7 mm, vias 0 -> 1
- net BUS0: track 0.64 -> 119.5 mm, vias 0 -> 1
- net Q: track 0.00 -> 116.2 mm
- net BUS1: track 0.00 -> 114.6 mm, vias 0 -> 1
- net BUS3: track 0.00 -> 109.2 mm, vias 0 -> 1
- net ~{MRD}: track 0.00 -> 102.3 mm
- net BUS2: track 0.64 -> 101.6 mm, vias 0 -> 1
- net BUS5: track 0.00 -> 100.0 mm, vias 0 -> 1
- net BUS7: track 0.00 -> 97.3 mm, vias 0 -> 1
- net INSEL: track 0.00 -> 97.0 mm, vias 0 -> 1
- net Net-(U4-Pad8): track 0.00 -> 96.5 mm, vias 0 -> 1
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- added copper zone on B.Cu, net GND
- added copper zone on F.Cu, net GND
Other:
- board text added: "0.1u"
- board text added: "00"
- board text added: "01"
- board text added: "02"
- board text added: "04"
- board text added: "08"
- board text added: "10K"
- board text added: "1802/MINI"
- board text added: "2"
- board text added: "22K"
- board text added: "3"
- board text added: "40"
- board text added: "4148"
- board text added: "50"
- board text added: "60"
- board text added: "70"
- board text added: "74HC00 QUAD NAND"
- board text added: "74HC04 HEX INVERTER"
- board text added: "74HC08 QUAD AND"
- board text added: "74HC11 TRIPLE AND"
- board text added: "74HC238 3-TO-8 DECODER"
- board text added: "74HC273 8-BIT REGISTER"
- board text added: "74HC4050 HEX BUFFER"
- board text added: "74HC573 OCTAL LATCH"
- board text added: "74HC74 DUAL D FLIP-FLOP"
- board text added: "80"
- board text added: "90"
- board text added: "A0"
- board text added: "ALL"
- board text added: "B0"
- board text added: "C0"
- board text added: "D0"
- board text added: "E0"
- board text added: "EF LINE"
- board text added: "F0"
- board text added: "I/O GROUP"
- board text added: "I/O PORT"
- board text added: "INPUT"
- board text added: "INT ENA"
- board text added: "JLCJLCJLCJLC"
- board text added: "JLCPCB ORDER #"
- board text added: "OUTPUT A"
- board text added: "OUTPUT B"
- board text added: "OUTPUTA"
- board text added: "OUTPUTB"
- board text added: "PARALLEL I/O"
- board text added: "SELECT"
- board text added: "rev A"

Commit message: Update to Rev B.
Connections:
- U1 pad 10: Net-(U1-Pad10) -> unconnected-(U1-Pad10)
- U1 pad 11: TPB -> GND
- U1 pad 13: INSEL -> /Ports/ISEL
- U1 pad 9: OUTSELA -> /Ports/OSEL
- U4 pad 12: Net-(U4-Pad12) -> /Ports/OSEL
- U4 pad 8: Net-(U4-Pad8) -> /Ports/ISEL
- U5 pad 11: Net-(U4-Pad12) -> /Ports/OSEL
- U7 pad 1: Net-(U4-Pad8) -> Net-(U7-Pad1)
- U8 pad 10: unconnected-(U8-Pad10) -> Net-(U7-Pad1)
- U8 pad 11: GND -> /Ports/ISEL
- U9 pad 3: Net-(U1-Pad10) -> TPB
Routing:
- net GND: track 507.9 -> 100.1 mm, vias 0 -> 1
- net /Ports/OSEL: track 0.00 -> 114.6 mm
- net Net-(U4-Pad8): track 96.5 -> 0.00 mm, vias 1 -> 0
- net Net-(U7-Pad1): track 0.00 -> 75.8 mm, vias 0 -> 1
- net /Ports/ISEL: track 0.00 -> 75.6 mm
- net Net-(U4-Pad12): track 47.9 -> 0.00 mm
- net INSEL: track 97.0 -> 52.3 mm, vias 1 -> 0
- net OUTSELA: track 70.5 -> 34.2 mm
- net Net-(U1-Pad10): track 35.2 -> 0.00 mm
- net Net-(D5-Pad1): track 64.2 -> 29.5 mm
- net BUS2: track 101.6 -> 127.1 mm
- net TPB: track 84.3 -> 61.9 mm
- net /Output Connectors/OUTA7: track 82.1 -> 103.4 mm, vias 1 -> 0
- net /Input Connector/STB: track 64.7 -> 83.7 mm, vias 1 -> 0
- net +5V: track 442.9 -> 426.5 mm, vias 0 -> 1
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Other:
- board text added: "rev B"
- board text removed: "rev A"
