File: 1802-Mini-PIO.kicad_sch (KiCad schematic)
At the start: 10 parts, among them J1 Mount, J10 OUT_PORTB, J2 Mount, J3 Mount, J4 Mount, J5 Expansion, J6 GRP_EXP, J7 GRP_SEL, J8 INP_PORT, J9 OUT_PORTA

Commit message: Update to Rev B.
Other:
- sheet Ports ports: added ISEL, OSEL; removed none
- sheet Service Request ports: added ISEL, OSEL; removed none
Changed lines of the file:
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@@
+    (stroke (width 0) (type default) (color 0 0 0 0))
+  )
+  (wire (pts (xy 19.05 86.36) (xy 30.48 86.36))
     (stroke (width 0) (type default) (color 0 0 0 0))
   )
@@
     (stroke (width 0) (type default) (color 0 0 0 0))
   )
+  (wire (pts (xy 19.05 133.35) (xy 19.05 86.36))
+    (stroke (width 0) (type default) (color 0 0 0 0))
+  )
   (wire (pts (xy 193.04 111.76) (xy 193.04 114.3))
     (stroke (width 0) (type default) (color 0 0 0 0))
@@
     (stroke (width 0) (type default) (color 0 0 0 0))
   )
+  (wire (pts (xy 25.4 92.71) (xy 30.48 92.71))
+    (stroke (width 0) (type default) (color 0 0 0 0))
+  )
   (wire (pts (xy 189.23 139.7) (xy 193.04 139.7))
     (stroke (width 0) (type default) (color 0 0 0 0))
@@
     (stroke (width 0) (type default) (color 0 0 0 0))
   )
+  (wire (pts (xy 31.75 133.35) (xy 19.05 133.35))
+    (stroke (width 0) (type default) (color 0 0 0 0))
+  )
   (wire (pts (xy 78.74 66.04) (xy 86.36 66.04))
     (stroke (width 0) (type default) (color 0 0 0 0))
@@
     (stroke (width 0) (type default) (color 0 0 0 0))
   )
+  (wire (pts (xy 25.4 127) (xy 25.4 92.71))
+    (stroke (width 0) (type default) (color 0 0 0 0))
+  )
   (wire (pts (xy 189.23 106.68) (xy 193.04 106.68))
     (stroke (width 0) (type default) (color 0 0 0 0))
@@
   )
   (wire (pts (xy 193.04 134.62) (xy 193.04 137.16))
+    (stroke (width 0) (type default) (color 0 0 0 0))
+  )
+  (wire (pts (xy 31.75 127) (xy 25.4 127))
     (stroke (width 0) (type default) (color 0 0 0 0))
   )
@@
       (effects (font (size 1.27 1.27)) (justify right))
     )
+    (pin "ISEL" output (at 31.75 127 180)
+      (effects (font (size 1.27 1.27)) (justify left))
+    )
+    (pin "OSEL" output (at 31.75 133.35 180)
+      (effects (font (size 1.27 1.27)) (justify left))
+    )
   )
   (sheet (at 30.48 35.56) (size 29.21 20.32) (fields_autoplaced)
@@
     (pin "STB" input (at 59.69 92.71 0)
       (effects (font (size 1.27 1.27)) (justify right))
+    )
+    (pin "ISEL" input (at 30.48 92.71 180)
+      (effects (font (size 1.27 1.27)) (justify left))
+    )
+    (pin "OSEL" input (at 30.48 86.36 180)
+      (effects (font (size 1.27 1.27)) (justify left))
     )
   )
@@
       (reference "U1") (unit 4) (value "74HC04") (footprint "Package_DIP:DIP-14_W7.62mm_Socket")
     )
-    (path "/9517ee2d-357d-4676-ab9b-c69e42f26ad4/c07a850f-51ae-44f0-a5ef-30de23c07a64"
+    (path "/88756d35-04bf-4708-813b-1e93de23b6c1/70c1a361-d99a-40fa-9649-72dd68555d79"
       (reference "U1") (unit 5) (value "74HC04") (footprint "Package_DIP:DIP-14_W7.62mm_Socket")
     )
@@
       (reference "U8") (unit 4) (value "74HC04") (footprint "Package_DIP:DIP-14_W7.62mm_Socket")
     )
-    (path "/88756d35-04bf-4708-813b-1e93de23b6c1/2253f74b-8671-4ce5-aed5-3a4639f87e07"
+    (path "/3ea2add1-0728-4c5b-b196-33ce47375e59/682a1fb7-ed1b-4588-b440-371e58c21d00"
       (reference "U8") (unit 5) (value "74HC04") (footprint "Package_DIP:DIP-14_W7.62mm_Socket")
     )
