File: ports.kicad_sch (KiCad schematic)
At the start: 5 parts, among them U1 74HC04, U4 74HC11, U5 74HC273, U6 74HC273, U7 74HC573

Commit message: Update to Rev B.
Parts:
- added U8: 74HC04, Package_DIP:DIP-14_W7.62mm_Socket, symbol 74xx:74HC04
Connections:
- net OSEL: now reaches U4.12, U5.11 (Cp)
- net at U7.1 (~{OE}): now also U8.10; no longer U4.8
- new net ISEL: U4.8, U8.11
Other:
- moved on the sheet: U4B, U4C
