File: service_request.kicad_sch (KiCad schematic)
At the start: 10 parts, among them U1 74HC04, U10 74HC08, U11 74HC74, U8 74HC04, U9 74HC74

Commit message: Update to Rev B.
Parts:
- removed unit 5 of U1
Connections:
- net TPB: now also U9.3 (C)
- net INSEL renamed ISEL
- net OUTSELA renamed OSEL
Changed lines of the file:
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@@
     (stroke (width 0) (type default) (color 0 0 0 0))
   )
-  (wire (pts (xy 41.91 60.96) (xy 52.07 60.96))
+  (wire (pts (xy 41.91 60.96) (xy 82.55 60.96))
     (stroke (width 0) (type default) (color 0 0 0 0))
   )
@@
   )
   (wire (pts (xy 205.74 58.42) (xy 205.74 62.23))
-    (stroke (width 0) (type default) (color 0 0 0 0))
-  )
-  (wire (pts (xy 67.31 60.96) (xy 82.55 60.96))
     (stroke (width 0) (type default) (color 0 0 0 0))
   )
@@
     )
   )
-  (global_label "INSEL" (shape input) (at 41.91 110.49 180) (fields_autoplaced)
-    (effects (font (size 1.27 1.27)) (justify right))
-    (property "Intersheet References" "${INTERSHEET_REFS}" (id 0) (at 34.2639 110.4106 0)
-      (effects (font (size 1.27 1.27)) (justify right) hide)
-    )
-  )
   (global_label "~{CLEAR}" (shape input) (at 41.91 125.73 180) (fields_autoplaced)
     (effects (font (size 1.27 1.27)) (justify right))
     (property "Intersheet References" "${INTERSHEET_REFS}" (id 0) (at 33.7801 125.6506 0)
-      (effects (font (size 1.27 1.27)) (justify right) hide)
-    )
-  )
-  (global_label "OUTSELA" (shape input) (at 41.91 44.45 180) (fields_autoplaced)
-    (effects (font (size 1.27 1.27)) (justify right))
-    (property "Intersheet References" "${INTERSHEET_REFS}" (id 0) (at 31.482 44.3706 0)
       (effects (font (size 1.27 1.27)) (justify right) hide)
     )
@@
     )
   )
+  (hierarchical_label "ISEL" (shape input) (at 41.91 110.49 180)
+    (effects (font (size 1.27 1.27)) (justify right))
+  )
+  (hierarchical_label "OSEL" (shape input) (at 41.91 44.45 180)
+    (effects (font (size 1.27 1.27)) (justify right))
+  )
   (hierarchical_label "SRA" (shape output) (at 139.7 55.88 0)
     (effects (font (size 1.27 1.27)) (justify left))
@@
     (pin "2")
   )
-  (symbol (lib_id "74xx:74HC04") (at 59.69 60.96 0) (unit 5)
-    (in_bom yes) (on_board yes) (fields_autoplaced)
-    (property "Reference" "U1" (id 0) (at 59.69 52.07 0))
-    (property "Value" "74HC04" (id 1) (at 59.69 54.61 0))
-    (property "Footprint" "Package_DIP:DIP-14_W7.62mm_Socket" (id 2) (at 59.69 60.96 0)
-      (effects (font (size 1.27 1.27)) hide)
-    )
-    (property "Datasheet" "https://assets.nexperia.com/documents/data-sheet/74HC_HCT04.pdf" (id 3) (at 59.69 60.96 0)
-      (effects (font (size 1.27 1.27)) hide)
-    )
-    (pin "1")
-    (pin "2")
-    (pin "3")
-    (pin "4")
-    (pin "5")
-    (pin "6")
-    (pin "8")
-    (pin "9")
-    (pin "10")
-    (pin "11")
-    (pin "12")
-    (pin "13")
-    (pin "14")
-    (pin "7")
-  )
   (symbol (lib_id "74xx:74HC04") (at 59.69 110.49 0) (unit 6)
